Commit message: test

File: src/inmoov_description/urdf/asmHand.urdf.xacro (robot description, xacro)
@@ -1,411 +1,505 @@
 <?xml version="1.0"?>
-<robot name="inmoov" xmlns:xacro="http://ros.org/wiki/xacro">
-<xacro:include filename="$(find inmoov_description)/urdf/materials.urdf.xacro" />
-<xacro:macro name="hand" params="side neg flip covers">
-  <link name="${side}_hand">
-    <visual>
-      <geometry>
-        <mesh filename="package://inmoov_meshes/meshes/${side}_hand.stl" scale="0.001 0.001 0.001"/>
-      </geometry>
-      <origin rpy="0 0 0" xyz="0 0 0"/>
-      <xacro:frame_color/>
-    </visual>
-  </link>
-  <link name="${side}_thumb1">
-    <visual>
-      <geometry>
-        <mesh filename="package://inmoov_meshes/meshes/${side}_thumb5_1.stl" scale="0.001 0.001 0.001"/>
-      </geometry>
-      <origin rpy="3.1415 0 0" xyz="0 0 0"/>
-      <xacro:frame_color/>
-    </visual>
-  </link>
-  <link name="${side}_thumb2">
-    <visual>
-      <geometry>
-        <mesh filename="package://inmoov_meshes/meshes/thumb5_2.stl" scale="0.001 0.001 0.001"/>
-      </geometry>
-      <origin rpy="0 0 3.1415" xyz="0 0 0"/>
-      <xacro:frame_color/>
-    </visual>
-  </link>
-  <link name="${side}_thumb3">
-    <visual>
-      <geometry>
-        <mesh filename="package://inmoov_meshes/meshes/thumb5_3.stl" scale="0.001 0.001 0.001"/>
-      </geometry>
-      <origin rpy="0 0 3.1415" xyz="0 0 0"/>
-      <xacro:frame_color/>
-    </visual>
-  </link>
-  <link name="${side}_index1">
-    <visual>
-      <geometry>
-        <mesh filename="package://inmoov_meshes/meshes/index3_1.stl" scale="0.001 0.001 0.001"/>
-      </geometry>
-      <origin rpy="0 0 3.1415" xyz="0 0 0"/>
-      <xacro:frame_color/>
-    </visual>
-  </link>
-  <link name="${side}_index2">
-    <visual>
-      <geometry>
-        <mesh filename="package://inmoov_meshes/meshes/index3_2.stl" scale="0.001 0.001 0.001"/>
-      </geometry>
-      <origin rpy="0 0 3.1415" xyz="0 0 0"/>
-      <xacro:frame_color/>
-    </visual>
-  </link>
-  <link name="${side}_index3">
-    <visual>
-      <geometry>
-        <mesh filename="package://inmoov_meshes/meshes/index3_3.stl" scale="0.001 0.001 0.001"/>
-      </geometry>
-      <origin rpy="0 0 3.1415" xyz="0 0 0"/>
-      <xacro:frame_color/>
-    </visual>
-  </link>
-  <link name="${side}_middle1">
-    <visual>
-      <geometry>
-        <mesh filename="package://inmoov_meshes/meshes/middle3_1.stl" scale="0.001 0.001 0.001"/>
-      </geometry>
-      <origin rpy="0 0 3.1415" xyz="0 0 0"/>
-      <xacro:frame_color/>
-    </visual>
-  </link>
-  <link name="${side}_middle2">
-    <visual>
-      <geometry>
-        <mesh filename="package://inmoov_meshes/meshes/middle3_2.stl" scale="0.001 0.001 0.001"/>
-      </geometry>
-      <origin rpy="0 0 3.1415" xyz="0 0 0"/>
-      <xacro:frame_color/>
-    </visual>
-  </link>
-  <link name="${side}_middle3">
-    <visual>
-      <geometry>
-        <mesh filename="package://inmoov_meshes/meshes/middle3_3.stl" scale="0.001 0.001 0.001"/>
-      </geometry>
-      <origin rpy="0 0 3.1415" xyz="0 0 0"/>
-      <xacro:frame_color/>
-    </visual>
-  </link>
-  <link name="${side}_ring1">
-    <visual>
-      <geometry>
-        <mesh filename="package://inmoov_meshes/meshes/${side}_ring3_1.stl" scale="0.001 0.001 0.001"/>
-      </geometry>
-      <origin rpy="0 0 3.1415" xyz="0 0 0"/>
-      <xacro:frame_color/>
-    </visual>
-  </link>
-  <link name="${side}_ring2">
-    <visual>
-      <geometry>
-        <mesh filename="package://inmoov_meshes/meshes/ring3_2.stl" scale="0.001 0.001 0.001"/>
-      </geometry>
-      <origin rpy="0 0 3.1415" xyz="0 0 0"/>
-      <xacro:frame_color/>
-    </visual>
-  </link>
-  <link name="${side}_ring3">
-    <visual>
-      <geometry>
-        <mesh filename="package://inmoov_meshes/meshes/ring3_3.stl" scale="0.001 0.001 0.001"/>
-      </geometry>
-      <origin rpy="0 0 3.1415" xyz="0 0 0"/>
-      <xacro:frame_color/>
-    </visual>
-  </link>
-  <link name="${side}_ring4">
-    <visual>
-      <geometry>
-        <mesh filename="package://inmoov_meshes/meshes/ring3_4.stl" scale="0.001 0.001 0.001"/>
-      </geometry>
-      <origin rpy="0 0 3.1415" xyz="0 0 0"/>
-      <xacro:frame_color/>
-    </visual>
-  </link>
-  <link name="${side}_pinky1">
-    <visual>
-      <geometry>
-        <mesh filename="package://inmoov_meshes/meshes/${side}_pinky3_1.stl" scale="0.001 0.001 0.001"/>
-      </geometry>
-      <origin rpy="0 0 3.1415" xyz="0 0 0"/>
-      <xacro:frame_color/>
-    </visual>
-  </link>
-  <link name="${side}_pinky2">
-    <visual>
-      <geometry>
-        <mesh filename="package://inmoov_meshes/meshes/pinky3_2.stl" scale="0.001 0.001 0.001"/>
-      </geometry>
-      <origin rpy="0 0 3.1415" xyz="0 0 0"/>
-      <xacro:frame_color/>
-    </visual>
-  </link>
-  <link name="${side}_pinky3">
-    <visual>
-      <geometry>
-        <mesh filename="package://inmoov_meshes/meshes/pinky3_3.stl" scale="0.001 0.001 0.001"/>
-      </geometry>
-      <origin rpy="0 0 3.1415" xyz="0 0 0"/>
-      <xacro:frame_color/>
-    </visual>
-  </link>
-  <link name="${side}_pinky4">
-    <visual>
-      <geometry>
-        <mesh filename="package://inmoov_meshes/meshes/pinky3_4.stl" scale="0.001 0.001 0.001"/>
-      </geometry>
-      <origin rpy="0 0 3.1415" xyz="0 0 0"/>
-      <xacro:frame_color/>
-    </visual>
-  </link>
-  <joint name="${side}_thumb1" type="revolute">
-   <axis xyz="0 0 1"/>
-   <limit effort="1000.0" lower="0" upper="${neg *1.57}" velocity="0.5"/>
-   <origin rpy="3.1415 ${neg * 0.1} 0" xyz="${neg * -0.029} 0 -0.0577"/>
-   <mimic joint="${side}_thumb" multiplier="${neg *-0.75}" offset="0"/>
-   <parent link="${side}_hand"/>
-   <child link="${side}_thumb1"/>
-  </joint>
-  <joint name="${side}_thumb" type="revolute">
-   <axis xyz="1 0 0"/>
-<limit effort="1000.0" lower="0" upper="1.5" velocity="0.5"/>
-    <origin rpy="0 ${neg * 2.3} ${neg * -0.3}" xyz="${neg * -0.02725} -0.0006 0.014"/>
-    <parent link="${side}_thumb1"/>
-    <child link="${side}_thumb2"/>
-  </joint>
-  <joint name="${side}_thumb3" type="revolute">
-   <axis xyz="1 0 0"/>
-<limit effort="1000.0" lower="-1.57" upper="0" velocity="0.5"/>
-<origin rpy="0 0 0" xyz="0 0 -0.035"/>
-    <mimic joint="${side}_thumb" multiplier="1" offset="0"/>
-    <parent link="${side}_thumb2"/>
-    <child link="${side}_thumb3"/>
-  </joint>
-  <joint name="${side}_index1" type="revolute">
-   <axis xyz="1 0 0"/>
-<limit effort="1000.0" lower="0" upper="1.5" velocity="0.5"/>
-<origin rpy="0 ${neg * -0.1} 3.1415" xyz="${neg * -0.0342} -0.0015 -0.119"/>
-    <mimic joint="${side}_index" multiplier="1" offset="0"/>
-    <parent link="${side}_hand"/>
-    <child link="${side}_index1"/>
-  </joint>
-  <joint name="${side}_index" type="revolute">
-   <axis xyz="1 0 0"/>
-<limit effort="1000.0" lower="0" upper="1.5" velocity="0.5"/>
-<origin rpy="0 0 0" xyz="0 0.001 -0.03595"/>
-    <parent link="${side}_index1"/>
-    <child link="${side}_index2"/>
-  </joint>
-  <joint name="${side}_index3" type="revolute">
-   <axis xyz="1 0 0"/>
-<limit effort="1000.0" lower="0" upper="1.5" velocity="0.5"/>
-<origin rpy="0 0 0" xyz="0 0 -0.024"/>
-    <mimic joint="${side}_index" multiplier="1" offset="0"/>
-    <parent link="${side}_index2"/>
-    <child link="${side}_index3"/>
-  </joint>
-  <joint name="${side}_middle1" type="revolute">
-   <axis xyz="1 0 0"/>
-<limit effort="1000.0" lower="0" upper="1.5" velocity="0.5"/>
-<origin rpy="0 0 3.1415" xyz="${neg * -0.007} -0.00175 -0.12325"/>
-    <mimic joint="${side}_middle" multiplier="1" offset="0"/>
-    <parent link="${side}_hand"/>
-    <child link="${side}_middle1"/>
-  </joint>
-  <joint name="${side}_middle" type="revolute">
-   <axis xyz="1 0 0"/>
-<limit effort="1000.0" lower="0" upper="1.5" velocity="0.5"/>
-<origin rpy="0 0 0" xyz="0 0.000 -0.0389"/>
-    <parent link="${side}_middle1"/>
-    <child link="${side}_middle2"/>
-  </joint>
-  <joint name="${side}_middle3" type="revolute">
-   <axis xyz="1 0 0"/>
-<limit effort="1000.0" lower="-1.57" upper="0" velocity="0.5"/>
-<origin rpy="0 0 0" xyz="0 0.0005 -0.0259"/>
-    <mimic joint="${side}_middle" multiplier="1" offset="0"/>
-    <parent link="${side}_middle2"/>
-    <child link="${side}_middle3"/>
-  </joint>
-  <joint name="${side}_ring1" type="revolute">
-   <axis xyz="0 0 1"/>
-<limit effort="1000.0" lower="${neg *-1.57}" upper="0" velocity="0.5"/>
-<origin rpy="0 ${neg * -0.7} 3.1415" xyz="${neg * 0.00705} 0 -0.0794"/>
-    <mimic joint="${side}_ring" multiplier="${neg * -0.1}" offset="0"/>
-    <parent link="${side}_hand"/>
-    <child link="${side}_ring1"/>
-  </joint>
-  <joint name="${side}_ring" type="revolute">
-   <axis xyz="1 0 0"/>
-<limit effort="1000.0" lower="0" upper="1.5" velocity="0.5"/>
-<origin rpy="0 ${neg * 0.7775} 0" xyz="${neg * -0.0351} 0.00126 -0.0166"/>
-    <parent link="${side}_ring1"/>
-    <child link="${side}_ring2"/>
-  </joint>
-  <joint name="${side}_ring3" type="revolute">
-   <axis xyz="1 0 0"/>
-<limit effort="1000.0" lower="-1.57" upper="0" velocity="0.5"/>
-<origin rpy="0 0 0" xyz="0 0.0005 -0.0345"/>
-    <mimic joint="${side}_ring" multiplier="1" offset="0"/>
-    <parent link="${side}_ring2"/>
-    <child link="${side}_ring3"/>
-  </joint>
-  <joint name="${side}_ring4" type="revolute">
-   <axis xyz="1 0 0"/>
-<limit effort="1000.0" lower="-1.57" upper="0" velocity="0.5"/>
-<origin rpy="0 0 0" xyz="0 0.0004 -0.0229"/>
-    <mimic joint="${side}_ring" multiplier="1" offset="0"/>
-    <parent link="${side}_ring3"/>
-    <child link="${side}_ring4"/>
-  </joint>
-  <joint name="${side}_pinky1" type="revolute">
-   <axis xyz="0 0 1"/>
-<limit effort="1000.0" lower="${neg *-1.57}" upper="0" velocity="0.5"/>
-<origin rpy="0 ${neg * -0.7} 3.1415" xyz="${neg * 0.0270} 0 -0.0555"/>
-    <mimic joint="${side}_pinky" multiplier="${neg * -0.1}" offset="0"/>
-    <parent link="${side}_hand"/>
-    <child link="${side}_pinky1"/>
-  </joint>
-  <joint name="${side}_pinky" type="revolute">
-   <axis xyz="1 0 0"/>
-<limit effort="1000.0" lower="0" upper="1.5" velocity="0.5"/>
-<origin rpy="0 ${neg * 0.93} 0" xyz="${neg * -0.046} -0 -0.0228"/>
-    <parent link="${side}_pinky1"/>
-    <child link="${side}_pinky2"/>
-  </joint>
-  <joint name="${side}_pinky3" type="revolute">
-   <axis xyz="1 0 0"/>
-<limit effort="1000.0" lower="-1.57" upper="0" velocity="0.5"/>
-<origin rpy="0 0 0" xyz="0 0.0005 -0.031"/>
-    <mimic joint="${side}_pinky" multiplier="1" offset="0"/>
-    <parent link="${side}_pinky2"/>
-    <child link="${side}_pinky3"/>
-  </joint>
-  <joint name="${side}_pinky4" type="revolute">
-   <axis xyz="1 0 0"/>
-<limit effort="1000.0" lower="-1.57" upper="0" velocity="0.5"/>
-<origin rpy="0 0 0" xyz="0 0.0004 -0.0208"/>
-    <mimic joint="${side}_pinky" multiplier="1" offset="0"/>
-    <parent link="${side}_pinky3"/>
-    <child link="${side}_pinky4"/>
-  </joint>
-  <link name="${side}_handcover">
-    <visual>
-      <geometry>
-        <mesh filename="package://inmoov_meshes/meshes/${side}_cover_hand.stl" scale="0.001 0.001 0.001"/>
-      </geometry>
-      <origin rpy="0 0 0" xyz="0 0 0"/>
-      <xacro:cover_color/>
-    </visual>
-  </link>
-  <link name="${side}_cover_handring">
-    <visual>
-      <geometry>
-        <mesh filename="package://inmoov_meshes/meshes/${side}_cover_handring.stl" scale="0.001 0.001 0.001"/>
-      </geometry>
-      <origin rpy="0 0 3.1415" xyz="0 0 0"/>
-      <xacro:cover_color/>
-    </visual>
-  </link>
-  <link name="${side}_cover_handpinky">
-    <visual>
-      <geometry>
-        <mesh filename="package://inmoov_meshes/meshes/${side}_cover_handpinky.stl" scale="0.001 0.001 0.001"/>
-      </geometry>
-      <origin rpy="0 0 3.1415" xyz="0 0 0"/>
-      <xacro:cover_color/>
-    </visual>
-  </link>
-  <link name="${side}_cover_thumb">
-    <visual>
-      <geometry>
-        <mesh filename="package://inmoov_meshes/meshes/${side}_cover_thumb.stl" scale="0.001 0.001 0.001"/>
-      </geometry>
-      <origin rpy="3.1415 0 0" xyz="0 0 0"/>
-      <xacro:cover_color/>
-    </visual>
-  </link>
-  <link name="${side}_cover_index">
-    <visual>
-      <geometry>
-        <mesh filename="package://inmoov_meshes/meshes/${side}_cover_index.stl" scale="0.001 0.001 0.001"/>
-      </geometry>
-      <origin rpy="0 0 3.1415" xyz="0 0 0"/>
-      <xacro:cover_color/>
-    </visual>
-  </link>
-  <link name="${side}_cover_middle">
-    <visual>
-      <geometry>
-        <mesh filename="package://inmoov_meshes/meshes/${side}_cover_middle.stl" scale="0.001 0.001 0.001"/>
-      </geometry>
-      <origin rpy="0 0 3.1415" xyz="0 0 0"/>
-      <xacro:cover_color/>
-    </visual>
-  </link>
-  <link name="${side}_cover_ring">
-    <visual>
-      <geometry>
-        <mesh filename="package://inmoov_meshes/meshes/${side}_cover_ring.stl" scale="0.001 0.001 0.001"/>
-      </geometry>
-      <origin rpy="0 0 3.1415" xyz="0 0 0"/>
-      <xacro:cover_color/>
-    </visual>
-  </link>
-  <link name="${side}_cover_pinky">
-    <visual>
-      <geometry>
-        <mesh filename="package://inmoov_meshes/meshes/${side}_cover_pinky.stl" scale="0.001 0.001 0.001"/>
-      </geometry>
-      <origin rpy="0 0 3.1415" xyz="0 0 0"/>
-      <xacro:cover_color/>
-    </visual>
-  </link>
-  <joint name="${side}_handcover" type="fixed">
-<origin rpy="0 0 0" xyz="${neg * -0.0192} 0.009 -0.0977"/>
-    <parent link="${side}_hand"/>
-    <child link="${side}_handcover"/>
-  </joint>
-  <joint name="${side}_cover_handring" type="fixed">
-<origin rpy="0 ${neg * 0.7} 0" xyz="${neg * -0.015} -0.009 -0.0008"/>
-    <parent link="${side}_ring1"/>
-    <child link="${side}_cover_handring"/>
-  </joint>
-  <joint name="${side}_cover_handpinky" type="fixed">
-<origin rpy="0 ${neg * 0.7} 0" xyz="${neg * -0.0205} -0.01 -0.0069"/>
-    <parent link="${side}_pinky1"/>
-    <child link="${side}_cover_handpinky"/>
-  </joint>
-  <joint name="${side}_cover_thumb" type="fixed">
-    <origin rpy="0 ${neg * 3.1} 0" xyz="${neg * -0.02125} -0.01 -0.0047"/>
-    <parent link="${side}_thumb1"/>
-    <child link="${side}_cover_thumb"/>
-  </joint>
-  <joint name="${side}_cover_index" type="fixed">
-    <origin rpy="${neg * 0.05} 0 0" xyz="0 -0.0071 -0.012"/>
-    <parent link="${side}_index1"/>
-    <child link="${side}_cover_index"/>
-  </joint>
-  <joint name="${side}_cover_middle" type="fixed">
-    <origin rpy="${neg * -0.05} 0 0" xyz="0 -0.0071 -0.012"/>
-    <parent link="${side}_middle1"/>
-    <child link="${side}_cover_middle"/>
-  </joint>
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
File: src/inmoov_description/urdf/asmHead.urdf.xacro (robot description, xacro)
@@ -2,6 +2,7 @@
 <robot name="inmoov" xmlns:xacro="http://ros.org/wiki/xacro">
 <xacro:include filename="$(find inmoov_description)/urdf/materials.urdf.xacro" />
+<xacro:include filename="$(find inmoov_description)/urdf/config.urdf.xacro" />
 <xacro:macro name="head" params="covers">
-  <link name="head_base">
+  <link name="head_base_link">
     <visual>
       <geometry>
@@ -12,5 +13,5 @@
     </visual>
   </link>
-  <link name="head">
+  <link name="head_link">
     <visual>
       <geometry>
@@ -21,14 +22,14 @@
     </visual>
   </link>
-  <link name="jaw">
+  <link name="jaw_link">
     <visual>
       <geometry>
         <mesh filename="package://inmoov_meshes/meshes/jaw.stl" scale="0.001 0.001 0.001"/>
       </geometry>
-      <origin rpy="0 0 3.1415" xyz="0 0 0"/>
+      <origin rpy="0 0 0" xyz="0 0 0"/>
       <xacro:cover_color/>
     </visual>
   </link>
-  <link name="skull">
+  <link name="skull_link">
     <visual>
       <geometry>
@@ -39,5 +40,5 @@
     </visual>
   </link>
-  <link name="left_ear">
+  <link name="left_ear_link">
     <visual>
       <geometry>
@@ -48,5 +49,5 @@
     </visual>
   </link>
-  <link name="right_ear">
+  <link name="right_ear_link">
     <visual>
       <geometry>
@@ -57,32 +58,32 @@
     </visual>
   </link>
-  <joint name="head_leftright" type="revolute">
+  <joint name="head_pan_joint" type="revolute">
    <axis xyz="0 0 1"/>
-   <limit effort="1000.0" lower="-1.57" upper="1.57" velocity="0.5"/>
+   <limit effort="1000.0" lower="${head_pan_joint_lower}" upper="${head_pan_joint_upper}" velocity="${head_pan_joint_velocity}" />
    <origin rpy="0 0 0" xyz="0 0 0.0245"/>
-   <parent link="head_base"/>
-   <child link="head"/>
+   <parent link="head_base_link"/>
+   <child link="head_link"/>
   </joint>
-  <joint name="jaw" type="revolute">
-   <axis xyz="1 0 0"/>
-   <limit effort="1000.0" lower="0" upper="0.15" velocity="0.5"/>
-   <origin rpy="0 -0.09 3.1415" xyz="0.0375 0.0005 0.0437"/>
-   <parent link="head"/>
-   <child link="jaw"/>
+  <joint name="jaw_joint" type="revolute">
+   <axis xyz="0 1 0"/>
+   <limit effort="1000.0" lower="${jaw_joint_lower}" upper="${jaw_joint_upper}" velocity="${jaw_joint_velocity}" />
+   <origin rpy="0 0.09 0" xyz="0.0375 0.0005 0.0437"/>
+   <parent link="head_link"/>
+   <child link="jaw_link"/>
   </joint>
-  <joint name="skull" type="fixed">
+  <joint name="skull_joint" type="fixed">
     <origin rpy="0 0 0" xyz="0.044 0 -0.0245"/>
-    <parent link="head"/>
-    <child link="skull"/>
+    <parent link="head_link"/>
+    <child link="skull_link"/>
   </joint>
-  <joint name="left_ear" type="fixed">
+  <joint name="left_ear_joint" type="fixed">
     <origin rpy="0 0 0" xyz="0.035 0.056 0.0437"/>
-    <parent link="head"/>
-    <child link="left_ear"/>
+    <parent link="head_link"/>
+    <child link="left_ear_link"/>
   </joint>
-  <joint name="right_ear" type="fixed">
+  <joint name="right_ear_joint" type="fixed">
     <origin rpy="0 0 0" xyz="0.035 -0.056 0.0437"/>
-    <parent link="head"/>
-    <child link="right_ear"/>
+    <parent link="head_link"/>
+    <child link="right_ear_link"/>
   </joint>
 </xacro:macro>

File: src/inmoov_description/urdf/asmTorso.urdf.xacro (robot description, xacro)
@@ -2,6 +2,7 @@
 <robot name="inmoov" xmlns:xacro="http://ros.org/wiki/xacro">
 <xacro:include filename="$(find inmoov_description)/urdf/materials.urdf.xacro" />
-<xacro:macro name="torso" params="side covers">
-  <link name="mid_stomach">
+<xacro:include filename="$(find inmoov_description)/urdf/config.urdf.xacro" />
+<xacro:macro name="torso" params="covers">
+  <link name="mid_stomach_link">
     <visual>
       <geometry>
@@ -12,5 +13,5 @@
     </visual>
   </link>
-  <link name="disk">
+  <link name="disk_link">
     <visual>
       <geometry>
@@ -21,5 +22,5 @@
     </visual>
   </link>
-  <link name="top_stomach">
+  <link name="top_stomach_link">
     <visual>
       <geometry>
@@ -30,5 +31,5 @@
     </visual>
   </link>
-  <link name="torso">
+  <link name="torso_link">
     <visual>
       <geometry>
@@ -48,4 +49,6 @@
     </visual>
   </link>
+    <link name="camera_link">
+   </link>
   <link name="kinect2_ir_optical_frame">
     <visual>
@@ -57,4 +60,8 @@
     </visual>
   </link>
+   <!-- <link name="camera_ir_optical_frame">
+  </link>
+   <link name="camera_rgb_optical_frame">
+    </link>-->
   <link name="kinect2_rgb_optical_frame">
     <visual>
@@ -66,5 +73,5 @@
     </visual>
   </link>
-  <link name="chestplate">
+  <link name="chestplate_link">
     <visual>
       <geometry>
@@ -75,43 +82,58 @@
     </visual>
   </link>
-  <joint name="waist_rotate" type="revolute">
+  <joint name="waist_pan_joint" type="revolute">
    <axis xyz="0 0 1"/>
-<limit effort="1000.0" lower="-1.57" upper="1.57" velocity="0.5"/>
-      <origin rpy="0 0 0" xyz="0 0 1.152"/>
-    <parent link="mid_stomach"/>
-    <child link="top_stomach"/>
+   <limit effort="1000.0" lower="${waist_pan_joint_lower}" upper="${waist_pan_joint_upper}" velocity="${waist_pan_joint_velocity}" />
+   <origin rpy="0 0 0" xyz="0 0 1.152"/>
+    <parent link="mid_stomach_link"/>
+    <child link="top_stomach_link"/>
   </joint>
-  <joint name="disk" type="fixed">
+  <joint name="disk_joint" type="fixed">
       <origin rpy="0 0 0" xyz="0.046 0 0.09"/>
-    <parent link="top_stomach"/>
-    <child link="disk"/>
+    <parent link="top_stomach_link"/>
+    <child link="disk_link"/>
   </joint>
-  <joint name="waist_lean" type="revolute">
+  <joint name="waist_roll_joint" type="revolute">
    <axis xyz="1 0 0"/>
-<limit effort="1000.0" lower="-0.30" upper="0.30" velocity="0.5"/>
-<origin rpy="0 0 0" xyz="0 0 0.11"/>
-    <parent link="top_stomach"/>
-    <child link="torso"/>
+   <limit effort="1000.0" lower="${waist_roll_joint_lower}" upper="${waist_roll_joint_upper}" velocity="${waist_roll_joint_velocity}" />
+   <origin rpy="0 0 0" xyz="0 0 0.11"/>
+    <parent link="top_stomach_link"/>
+    <child link="torso_link"/>
   </joint>
-  <joint name="chestplate" type="fixed">
-<origin rpy="0 0 0" xyz="0.039 0 0.025"/>
-    <parent link="torso"/>
-    <child link="chestplate"/>
+  <joint name="chestplate_joint" type="fixed">
+<origin rpy="0 0 0" xyz="0.042 0 0.025"/>
+    <parent link="torso_link"/>
+    <child link="chestplate_link"/>
   </joint>
-  <joint name="kinect2" type="fixed">
+  <joint name="kinect2_joint" type="fixed">
 <origin rpy="-1.57 0 -1.57" xyz="0 0 0.066"/>
-    <parent link="torso"/>
+    <parent link="torso_link"/>
     <child link="kinect2_link"/>
   </joint>
-  <joint name="kinect2_ir_optical_frame" type="fixed">
+    <joint name="camera_joint" type="fixed">
+<origin rpy="0 .7243116 0" xyz="0.03 0 .1921"/>
+    <parent link="chestplate_link"/>
+    <child link="camera_link"/>
+  </joint>
+  <joint name="kinect2_ir_optical_frame_joint" type="fixed">
 <origin rpy="-1.57 0 -1.57" xyz="0 0 0.066"/>
-    <parent link="torso"/>
+    <parent link="torso_link"/>
     <child link="kinect2_ir_optical_frame"/>
   </joint>
-  <joint name="kinect2_rgb_optical" type="fixed">
+ <!--<joint name="camera_ir_optical_frame_joint" type="fixed">
+<origin rpy="-2.3553 0 -1.57" xyz="1 1 1"/>
+    <parent link="camera_link"/>
+    <child link="camera_ir_optical_frame"/>
+  </joint>-->
+  <joint name="kinect2_rgb_optical_joint" type="fixed">
 <origin rpy="-1.57 0 -1.57" xyz="0 0 0.066"/>
-    <parent link="torso"/>
+    <parent link="torso_link"/>
     <child link="kinect2_rgb_optical_frame"/>
   </joint>
+ <!-- <joint name="camera_rgb_optical_joint" type="fixed">
+<origin rpy="-2.3553 0 -1.57" xyz=" 1 1 1"/>
+    <parent link="camera_link"/>
+    <child link="camera_rgb_optical_frame"/>
+  </joint>-->
 </xacro:macro>
 </robot>
